File: Starter/Starter.kicad_pcb (KiCad board)
At the start: 2 copper layers, 139.7 x 72.5 mm, 60 parts, among them J2 Speaker, J5 Conn_01x08_Pin, M1 Vibration Motor, Q1 2N2222, SW1 UP, SW2 LEFT, SW3 DOWN, SW4 RIGHT, U2 LP-MSPM0G3507, U3 MCP34119D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

Commit message: final board! ordered
Parts:
- removed J5: Conn_01x08_Pin, Connector_PinSocket_2.54mm:PinSocket_1x08_P2.54mm_Vertical
- R11, R4, R6, R7, R9: moved to B.Cu
- moved R6 32.0 mm to (127.5, 73.8)
- moved R4 29.8 mm to (127.5, 75.5)
- moved R11 27.8 mm to (127.5, 77.2)
- moved R9 26.2 mm to (127.5, 79.0)
- moved R7 24.9 mm to (127.5, 80.8)
- moved R18 9.65 mm to (159.2, 80.0)
- turned C14 to 180 degrees
- turned C15 to 0 degrees
Routing:
- net /PB18: track 0.00 -> 93.5 mm, vias 0 -> 1
- net /DAC0: track 0.00 -> 87.7 mm, vias 0 -> 4
- net /PA17: track 0.00 -> 80.5 mm
- net /MTR_PWM: track 0.00 -> 70.6 mm, vias 0 -> 1
- net /SPI_MOSI: track 0.00 -> 65.8 mm
- net /PA18: track 0.00 -> 64.3 mm
- net /SPI_MISO: track 0.00 -> 64.1 mm
- net /UART2_RX: track 0.00 -> 63.7 mm
- net Net-(D4-K): track 0.00 -> 61.3 mm, vias 0 -> 2
- net Net-(D3-A): track 0.00 -> 60.7 mm, vias 0 -> 3
- net /SDC_CS: track 0.00 -> 57.4 mm
- net Net-(D2-A): track 0.00 -> 57.0 mm, vias 0 -> 3
- net Net-(D6-A): track 0.00 -> 56.7 mm, vias 0 -> 3
- net /TFT_CS: track 0.00 -> 54.4 mm, vias 0 -> 1
- net /SPI_SCK: track 0.00 -> 54.0 mm
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- added copper zone on In2.Cu, net +3V3
- added copper zone on In2.Cu, net +5V
- added copper zone on In1.Cu, net GND
Other:
- copper layers 2 -> 4
- board text added: "Ravi Shah Alice Di Mauro"
